File: ewod_10bus.kicad_sch (KiCad schematic)
At the start: 41 parts, among them J1 B2P-VH, J2 B2P-VH, J3 B2P-VH, J4 B2P-VH, J5 B2P-VH, J6 B2P-VH, J7 B2P-VH, J8 Barrel_Jack, J9 031-5637, K1 AQV254A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

Commit message: One More
Parts:
- removed C1: 10 uF, Capacitor_SMD:C_0805_2012Metric, symbol Device:C
- removed C2: EEU-FR1A221, Capacitor_THT:CP_Radial_D6.3mm_P2.50mm, symbol SamacSys_Parts:EEU-FR1A221
- removed C4: 0.1 uF, Capacitor_SMD:C_0805_2012Metric, symbol Device:C
- removed C6: 100n, Capacitor_SMD:C_0603_1608Metric, symbol Device:C
